Commit message: starting to build the gazebo world and added pulgin of lidar

File: all_descriptions/lidar_description/urdf/hokuyo.urdf.xacro (robot description, xacro)
@@ -24,5 +24,5 @@
             </inertial>
         </link>
-        <joint name="hokuyo_joint" type="fixed">
+        <joint name="laser_joint" type="fixed">
             <axis xyz="0 0 1" />
             <origin xyz="0 0 0.035" rpy="0 0 0"/>
@@ -30,4 +30,27 @@
             <child link="laser"/>
         </joint>
+        <gazebo reference="laser">
+            <sensor:ray name="laser">
+                <rayCount>180</rayCount>
+                <rangeCount>180</rangeCount>
+                <laserCount>1</laserCount>
+                <origin>0.0 0.0 0.0</origin>
+                <displayRays>false</displayRays>
+                <minAngle>-130</minAngle>
+                <maxAngle>130</maxAngle>
+                <minRange>0.08</minRange>
+                <maxRange>10.0</maxRange>
+                <resRange>0.01</resRange>
+                <updateRate>20</updateRate>
+                <controller:gazebo_ros_laser name="gazebo_ros_laser_controller" plugin="libgazebo_ros_laser.so">
+                    <gaussianNoise>0.005</gaussianNoise>
+                    <alwaysOn>true</alwaysOn>
+                    <updateRate>20</updateRate>
+                    <topicName>scan</topicName>
+                    <frameName>laser</frameName>
+                    <interface:laser name="gazebo_ros_laser_iface" />
+                </controller:gazebo_ros_laser>
+            </sensor:ray>
+        </gazebo>
     </xacro:macro>
 </robot>

Commit message: debugging the simulation

File: all_descriptions/lidar_description/urdf/hokuyo.urdf.xacro (robot description, xacro)
@@ -30,27 +30,29 @@
             <child link="laser"/>
         </joint>
-        <gazebo reference="laser">
-            <sensor:ray name="laser">
-                <rayCount>180</rayCount>
-                <rangeCount>180</rangeCount>
-                <laserCount>1</laserCount>
-                <origin>0.0 0.0 0.0</origin>
-                <displayRays>false</displayRays>
-                <minAngle>-130</minAngle>
-                <maxAngle>130</maxAngle>
-                <minRange>0.08</minRange>
-                <maxRange>10.0</maxRange>
-                <resRange>0.01</resRange>
-                <updateRate>20</updateRate>
-                <controller:gazebo_ros_laser name="gazebo_ros_laser_controller" plugin="libgazebo_ros_laser.so">
-                    <gaussianNoise>0.005</gaussianNoise>
-                    <alwaysOn>true</alwaysOn>
+        <!-- <xacro:macro name="turtlebot_sim_laser"> -->
+            <!-- <gazebo reference="laser">
+                <sensor:ray name="laser">
+                    <rayCount>180</rayCount>
+                    <rangeCount>180</rangeCount>
+                    <laserCount>1</laserCount>
+                    <origin>0.0 0.0 0.0</origin>
+                    <displayRays>false</displayRays>
+                    <minAngle>-130</minAngle>
+                    <maxAngle>130</maxAngle>
+                    <minRange>0.08</minRange>
+                    <maxRange>10.0</maxRange>
+                    <resRange>0.01</resRange>
                     <updateRate>20</updateRate>
-                    <topicName>scan</topicName>
-                    <frameName>laser</frameName>
-                    <interface:laser name="gazebo_ros_laser_iface" />
-                </controller:gazebo_ros_laser>
-            </sensor:ray>
-        </gazebo>
+                    <controller:gazebo_ros_laser name="gazebo_ros_laser_controller" plugin="libgazebo_ros_laser.so">
+                        <gaussianNoise>0.005</gaussianNoise>
+                        <alwaysOn>true</alwaysOn>
+                        <updateRate>20</updateRate>
+                        <topicName>/scan</topicName>
+                        <frameName>laser</frameName>
+                        <interface:laser name="gazebo_ros_laser_iface" />
+                    </controller:gazebo_ros_laser>
+                </sensor:ray>
+            </gazebo> -->
+        <!-- </xacro:macro> -->
     </xacro:macro>
 </robot>

File: all_descriptions/tgrip_description/urdf/tgrip.urdf.xacro (robot description, xacro)
@@ -2,12 +2,15 @@
 <robot name="tgrip" xmlns:xacro="http://ros.org/wiki/xacro">
   <xacro:include filename="$(find turtlebot_description)/urdf/turtlebot_common_library.urdf.xacro" />
+  <xacro:include filename="$(find kobuki_description)/urdf/kobuki.urdf.xacro" />
   <xacro:include filename="$(find turtlebot_description)/urdf/stacks/hexagons.urdf.xacro"/>
   <xacro:include filename="$(find turtlebot_description)/urdf/sensors/kinect.urdf.xacro"/>
-  <xacro:include filename="$(find kinect_description)/urdf/kinect.urdf.xacro"/>
+  <!-- <xacro:include filename="$(find kinect_description)/urdf/kinect.urdf.xacro"/>
   <xacro:include filename="$(find lidar_description)/urdf/hokuyo.urdf.xacro"/>
-  <xacro:include filename="$(find kobuki_description)/urdf/kobuki.urdf.xacro" />
+  <xacro:include filename="$(find lidar_description)/urdf/hokuyo.gazebo" />
+  <xacro:include filename="$(find kobuki_description)/urdf/kobuki_gazebo.urdf.xacro" />
+  <xacro:include filename="$(find tgrip_description)/urdf/tgrip.gazebo" /> -->
   <kobuki/>
   <stack_hexagons parent="base_link"/>
-  <xacro:sensor_kinect parent="base_footprint" cam_px="0.03" cam_pz="0.3" cam_or="3.14" cam_op="0.475" cam_oy="0"/>
-  <xacro:sensor_hokuyo parent="plate_top_link"/>
+  <!-- <xacro:sensor_kinect parent="base_footprint" cam_px="0.03" cam_pz="0.3" cam_or="3.14" cam_op="0.475" cam_oy="0"/>
+  <xacro:sensor_hokuyo parent="plate_top_link"/> -->
 </robot>
