Commit message: manipulation module, 1st commit, made 3 actionlib related packages, imported 2 om packages, and changed the urdf files.

File: all_descriptions/openmanipulator_description/urdf/open_manipulator_workspace.urdf.xacro (robot description, xacro)
@@ -1,34 +1,35 @@
 <?xml version="1.0"?>
 <!-- Open_Manipulator Chain -->
-<robot xmlns:xacro="http://ros.org/wiki/xacro">
-  <!-- Link 1 -->
-  <link name="workspace">
-    <visual>
-      <origin xyz="-0.2 0 -0.15" rpy="0 0 0"/>
-      <geometry>
-        <mesh filename="package://om_test/urdf/work_space.stl" scale="0.001 0.001 0.001"/>
-      </geometry>
-      <material name="grey"/>
-    </visual>
-    <collision>
-      <origin xyz="-0.2 0 -0.15" rpy="0 0 0"/>
-      <geometry>
-        <mesh filename="package://om_test/urdf/work_space.stl" scale="0.001 0.001 0.001"/>
-      </geometry>
-    </collision>
-    <inertial>
-      <origin xyz="3.0876154e-04 0.0000000e+00 -1.2176461e-04" />
-      <mass value="7.9119962e-02" />
-      <inertia ixx="1.2505234e-05" ixy="0.0" ixz="-1.7855208e-07"
-               iyy="2.1898364e-05" iyz="0.0"
-               izz="1.9267361e-05" />
-    </inertial>
-  </link>
-  <!-- Joint 1 -->
-  <joint name="workspace" type="fixed">
-    <parent link="workspace"/>
-    <child link="link1"/>
-    <origin xyz="0.0 0.0 0.0" rpy="0 0 0"/>
-    <axis xyz="0 0 1"/>
-  </joint>
+<robot name ="workspace" xmlns:xacro="http://ros.org/wiki/xacro">
+  <xacro:macro name="workspace" params="parent ">
+    <!-- Link 1 -->
+    <link name="workspace">
+      <visual>
+        <origin xyz="0.18 0.2 0" rpy="0 0 ${-pi/2}"/>
+        <geometry>
+          <mesh filename="package://om_test/urdf/work_space.stl" scale="0.001 0.001 0.001"/>
+        </geometry>
+        <material name="grey"/>
+      </visual>
+      <collision>
+        <origin xyz="0.18 0.2 0" rpy="0 0 ${-pi/2}"/>
+        <geometry>
+          <mesh filename="package://om_test/urdf/work_space.stl" scale="0.001 0.001 0.001"/>
+        </geometry>
+      </collision>
+      <inertial>
+        <origin xyz="3.0876154e-04 0.0000000e+00 -1.2176461e-04" />
+        <mass value="7.9119962e-02" />
+        <inertia ixx="1.2505234e-05" ixy="0.0" ixz="-1.7855208e-07"
+                iyy="2.1898364e-05" iyz="0.0"
+                izz="1.9267361e-05" />
+      </inertial>
+    </link>
+    <joint name="workspace" type="fixed">
+      <parent link="${parent}"/>
+      <child link="workspace"/>
+      <origin xyz="0.0 0.0 0.0" rpy="0 0 0"/>
+      <axis xyz="0 0 1"/>
+    </joint>
+  </xacro:macro>
 </robot>

File: all_descriptions/tgrip_description/urdf/tgrip.urdf.xacro (robot description, xacro)
@@ -7,7 +7,19 @@
   <xacro:include filename="$(find lidar_description)/urdf/hokuyo.urdf.xacro"/>
   <xacro:include filename="$(find kobuki_description)/urdf/kobuki.urdf.xacro" />
-  <kobuki/>
-  <stack_hexagons parent="base_link"/>
   <xacro:sensor_kinect parent="base_footprint" cam_px="0.03" cam_pz="0.3" cam_or="3.14" cam_op="0.475" cam_oy="0"/>
   <xacro:sensor_hokuyo parent="plate_top_link"/>
+  <!-- Import manip -->
+  <xacro:include filename="$(find open_manipulator_description)/urdf/open_manipulator_robot.urdf.xacro"/>
+  <!-- Import work space -->
+  <xacro:include filename="$(find openmanipulator_description)/urdf/open_manipulator_workspace.urdf.xacro" />
+  <!-- World fixed joint-->
+  <joint name="fix_world" type="fixed">
+    <origin xyz="0.16 -0.08 0.14" rpy="0 0 ${-pi/2}"/>
+    <parent link="base_link"/>
+    <child link="world"/>
+  </joint>
+  <!-- Workspace joint-->
+  <workspace parent="base_link"/>
+  <stack_hexagons parent="base_link"/>
+  <!-- <kobuki/> -->
 </robot>

Commit message: Improved the robot_description. I decoupled the openmanipulator_description pacakge with the om_test. And I create view_model.rviz for a quicker visualization.

File: all_descriptions/openmanipulator_description/urdf/open_manipulator_workspace.urdf.xacro (robot description, xacro)
@@ -8,5 +8,5 @@
         <origin xyz="0.18 0.2 0" rpy="0 0 ${-pi/2}"/>
         <geometry>
-          <mesh filename="package://om_test/urdf/work_space.stl" scale="0.001 0.001 0.001"/>
+          <mesh filename="package://openmanipulator_description/mesh/work_space.stl" scale="0.001 0.001 0.001"/>
         </geometry>
         <material name="grey"/>
@@ -15,5 +15,5 @@
         <origin xyz="0.18 0.2 0" rpy="0 0 ${-pi/2}"/>
         <geometry>
-          <mesh filename="package://om_test/urdf/work_space.stl" scale="0.001 0.001 0.001"/>
+          <mesh filename="package://openmanipulator_description/mesh/work_space.stl" scale="0.001 0.001 0.001"/>
         </geometry>
       </collision>

Commit message: optimized the tgrip_nav_srvcli for gmapping and amcl for both sim and real world.

File: all_descriptions/openmanipulator_description/urdf/open_manipulator_workspace.urdf.xacro (robot description, xacro)
@@ -12,10 +12,4 @@
         <material name="grey"/>
       </visual>
-      <collision>
-        <origin xyz="0.18 0.2 0" rpy="0 0 ${-pi/2}"/>
-        <geometry>
-          <mesh filename="package://openmanipulator_description/mesh/work_space.stl" scale="0.001 0.001 0.001"/>
-        </geometry>
-      </collision>
       <inertial>
         <origin xyz="3.0876154e-04 0.0000000e+00 -1.2176461e-04" />

File: all_descriptions/tgrip_description/urdf/tgrip.urdf.xacro (robot description, xacro)
@@ -4,7 +4,8 @@
   <xacro:include filename="$(find turtlebot_description)/urdf/stacks/hexagons.urdf.xacro"/>
   <xacro:include filename="$(find turtlebot_description)/urdf/sensors/kinect.urdf.xacro"/>
+  <xacro:include filename="$(find kobuki_description)/urdf/kobuki.urdf.xacro" />
   <xacro:include filename="$(find kinect_description)/urdf/kinect.urdf.xacro"/>
+  <xacro:include filename="$(find lidar_description)/urdf/hokuyo.gazebo"/>
   <xacro:include filename="$(find lidar_description)/urdf/hokuyo.urdf.xacro"/>
-  <xacro:include filename="$(find kobuki_description)/urdf/kobuki.urdf.xacro" />
   <!--stack_hexagons parent="base_footprint"/-->
   <xacro:sensor_kinect parent="base_footprint" cam_px="0.03" cam_pz="0.3" cam_or="3.14" cam_op="0.475" cam_oy="0"/>

Commit message: Deleted intertia of the om workspace, which should be 0 weight. And I added color to the material tag, trying to make it transparent, but failed.

File: all_descriptions/openmanipulator_description/urdf/open_manipulator_workspace.urdf.xacro (robot description, xacro)
@@ -1,5 +1,6 @@
 <?xml version="1.0"?>
 <!-- Open_Manipulator Chain -->
-<robot name ="workspace" xmlns:xacro="http://ros.org/wiki/xacro">
+<robot name ="workspace"
+  xmlns:xacro="http://ros.org/wiki/xacro">
   <xacro:macro name="workspace" params="parent ">
     <!-- Link 1 -->
@@ -10,13 +11,8 @@
           <mesh filename="package://openmanipulator_description/mesh/work_space.stl" scale="0.001 0.001 0.001"/>
         </geometry>
-        <material name="grey"/>
+        <material name="grey">
+          <color rgba="0.5 0.5 0.5 0.2"/>
+        </material>
       </visual>
-      <inertial>
-        <origin xyz="3.0876154e-04 0.0000000e+00 -1.2176461e-04" />
-        <mass value="7.9119962e-02" />
-        <inertia ixx="1.2505234e-05" ixy="0.0" ixz="-1.7855208e-07"
-                iyy="2.1898364e-05" iyz="0.0"
-                izz="1.9267361e-05" />
-      </inertial>
     </link>
     <joint name="workspace" type="fixed">
