Commit message: deletedf the geometry tag of the middle plate and the sensore pole, which we don't use.

File: all_descriptions/openmanipulator_description/urdf/hexagons.urdf.xacro (robot description, xacro)
@@ -102,7 +102,7 @@
       <visual>
         <origin xyz="0 0 -0.01" rpy="0 0 0"/>
-        <geometry>
+        <!-- <geometry>
           <mesh filename="package://turtlebot_description/meshes/sensors/sensor_pole.dae" />
-        </geometry>
+        </geometry> -->
       </visual>
       <collision>
@@ -171,7 +171,7 @@
       <visual>
         <origin xyz="0 0 0" rpy="0 0 0"/>
-        <geometry>
-          <mesh filename="package://turtlebot_description/meshes/stacks/hexagons/plate_middle.dae"/>
-        </geometry>
+        <!-- <geometry> -->
+          <!-- <mesh filename="package://turtlebot_description/meshes/stacks/hexagons/plate_middle.dae"/> -->
+        <!-- </geometry> -->
       </visual>
       <!-- <collision>

Commit message: open manipulator description update

File: all_descriptions/openmanipulator_description/urdf/hexagons.urdf.xacro (robot description, xacro)
@@ -102,7 +102,7 @@
       <visual>
         <origin xyz="0 0 -0.01" rpy="0 0 0"/>
-        <!-- <geometry>
+        <geometry>
           <mesh filename="package://turtlebot_description/meshes/sensors/sensor_pole.dae" />
-        </geometry> -->
+        </geometry>
       </visual>
       <collision>
@@ -163,5 +163,5 @@
     <stack_middle_pole parent="${parent}" number="2" x_loc="-0.0381" y_loc= "0.1505" z_loc="0.1640"/>
     <stack_middle_pole parent="${parent}" number="3" x_loc="-0.0381" y_loc="-0.1505" z_loc="0.1640"/>
-    <joint name="plate_middle_joint" type="fixed">
+    <!-- <joint name="plate_middle_joint" type="fixed">
       <origin xyz="-0.01364 0.0 0.1874" rpy="0 0 0"/>
       <parent link="${parent}"/>
@@ -171,14 +171,14 @@
       <visual>
         <origin xyz="0 0 0" rpy="0 0 0"/>
-        <!-- <geometry> -->
-          <!-- <mesh filename="package://turtlebot_description/meshes/stacks/hexagons/plate_middle.dae"/> -->
-        <!-- </geometry> -->
-      </visual>
-      <!-- <collision>
+        <geometry>
+          <mesh filename="package://turtlebot_description/meshes/stacks/hexagons/plate_middle.dae"/>
+        </geometry>
+      </visual>
+      <collision>
         <origin xyz="0.01364 0.0 0.0" rpy="0 0 0"/>
         <geometry>
           <cylinder length="0.006" radius="0.170"/>
         </geometry>
-      </collision> -->
+      </collision>
       <inertial>
         <mass value="0.520" />
@@ -188,5 +188,5 @@
                  izz="0.006656" />
       </inertial>
-    </link>
+    </link> -->
     <stack_top_pole parent="${parent}" number="0" x_loc= "0.0381" y_loc= "0.1505" z_loc="0.2920"/>
     <stack_top_pole parent="${parent}" number="1" x_loc= "0.0381" y_loc="-0.1505" z_loc="0.2920"/>

File: all_descriptions/tgrip_description/urdf/tgrip.urdf.xacro (robot description, xacro)
@@ -19,5 +19,5 @@
   <!-- World fixed joint-->
   <joint name="fix_world" type="fixed">
-    <origin xyz="0.16 -0.08 0.17" rpy="0 0 ${-pi/2}"/>
+    <origin xyz="0.16 -0.08 0.15" rpy="0 0 ${-pi/2}"/>
     <parent link="base_footprint"/>
     <child link="link1"/>

File: open_manipulator/open_manipulator_description/urdf/open_manipulator.urdf.xacro (robot description, xacro)
@@ -219,5 +219,5 @@
   </joint>
   <!-- end effector link -->
-  <!-- <link name="end_effector_link">
+  <link name="end_effector_link">
     <visual>
       <origin xyz="0 0 0" rpy="0 0 0"/>
@@ -234,5 +234,5 @@
                izz="1.0e-03" />
     </inertial>
-  </link> -->
+  </link>
   <!-- Realsense Camera Joint Position -->
   <!-- <joint name="camera_joint" type="fixed">
