Commit message: fixed the joints of the om in gazebo to solve issue #2

File: all_descriptions/openmanipulator_description/urdf/open_manipulator_nav.urdf.xacro (robot description, xacro)
@@ -26,5 +26,5 @@
   </link>
   <!-- Joint 1 -->
-  <joint name="joint1" type="revolute">
+  <joint name="joint1" type="fixed">
     <parent link="link1"/>
     <child link="link2"/>
@@ -57,5 +57,5 @@
   </link>
   <!--  Joint 2 -->
-  <joint name="joint2" type="revolute">
+  <joint name="joint2" type="fixed">
     <parent link="link2"/>
     <child link="link3"/>
@@ -88,5 +88,5 @@
   </link>
   <!--  Joint 3 -->
-  <joint name="joint3" type="revolute">
+  <joint name="joint3" type="fixed">
     <parent link="link3"/>
     <child link="link4"/>
@@ -119,5 +119,5 @@
   </link>
   <!--  Joint 4 -->
-  <joint name="joint4" type="revolute">
+  <joint name="joint4" type="fixed">
     <parent link="link4"/>
     <child link="link5"/>
@@ -150,5 +150,5 @@
   </link>
   <!--  Gripper joint -->
-  <joint name="gripper" type="prismatic">
+  <joint name="gripper" type="fixed">
     <parent link="link5"/>
     <child link="gripper_link"/>
@@ -181,5 +181,5 @@
   </link>
   <!--  Gripper joint sub -->
-  <joint name="gripper_sub" type="prismatic">
+  <joint name="gripper_sub" type="fixed">
     <parent link="link5"/>
     <child link="gripper_link_sub"/>

File: all_descriptions/tgrip_description/urdf/tgrip.urdf.xacro (robot description, xacro)
@@ -12,9 +12,9 @@
   <xacro:include filename="$(find open_manipulator_description)/urdf/materials.xacro" />
   <!-- Import all Gazebo-customization elements, including Gazebo colors -->
-  <xacro:include filename="$(find open_manipulator_description)/urdf/open_manipulator.gazebo.xacro" />
+  <!-- <xacro:include filename="$(find open_manipulator_description)/urdf/open_manipulator.gazebo.xacro" /> -->
   <!-- Import Transmission -->
   <xacro:include filename="$(find open_manipulator_description)/urdf/open_manipulator.transmission.xacro" />
   <!-- Import URDF -->
-  <xacro:include filename="$(find open_manipulator_description)/urdf/open_manipulator.urdf.xacro" />
+  <!-- <xacro:include filename="$(find open_manipulator_description)/urdf/open_manipulator.urdf.xacro" /> -->
   <!-- World fixed joint-->
   <joint name="fix_world" type="fixed">
@@ -25,6 +25,6 @@
   <!-- Import manip -->
 <!-- for nav module -->
-  <!-- <xacro:include filename="$(find openmanipulator_description)/urdf/open_manipulator_nav.urdf.xacro" /> -->
-  <!-- <xacro:include filename="$(find open_manipulator_description)/urdf/open_manipulator.gazebo.xacro" /> -->
+  <xacro:include filename="$(find openmanipulator_description)/urdf/open_manipulator_nav.urdf.xacro" />
+  <xacro:include filename="$(find openmanipulator_description)/urdf/open_manipulator_nav.gazebo.xacro" />
 <!-- for nav module -->
   <!-- Import work space -->
