Commit message: Calibration joint for kinect
Added a floating joint(6DOF) to the tgrip.urdf.xacro file that can be used for the calibration of kinect relative to the open manipulator.
The joint kinect_adjust connects kinect to the base_footprint through link kinect_adjust_link (previously kinect as connected directly to base_footprint)
Note that gui isn't automatically enabled in rviz.

File: all_descriptions/tgrip_description/urdf/tgrip.urdf.xacro (robot description, xacro)
@@ -9,5 +9,12 @@
   <xacro:include filename="$(find lidar_description)/urdf/hokuyo.urdf.xacro"/>
   <!--stack_hexagons parent="base_footprint"/-->
-  <xacro:sensor_kinect parent="base_footprint" cam_px="0.03" cam_pz="0.3" cam_or="3.14" cam_op="0.475" cam_oy="0"/>
+  <link name="kinect_adjust_link"/>
+  <joint name="kinect_adjust" type="floating">
+    <origin xyz="0 0 0" rpy="0 0 0"/>
+    <parent link="base_footprint"/>
+    <child link="kinect_adjust_link"/>
+    <limit effort="10" lower="-0.2" upper="0.2"/>
+  </joint>
+  <xacro:sensor_kinect parent="kinect_adjust" cam_px="0.03" cam_pz="0.3" cam_or="3.14" cam_op="0.475" cam_oy="0"/>
   <xacro:sensor_hokuyo parent="plate_top_link"/>
   <!-- Import manip -->

Commit message: Commented out the kinect adjust joint to prevent parsing error

File: all_descriptions/tgrip_description/urdf/tgrip.urdf.xacro (robot description, xacro)
@@ -9,5 +9,5 @@
   <xacro:include filename="$(find lidar_description)/urdf/hokuyo.urdf.xacro"/>
   <!--stack_hexagons parent="base_footprint"/-->
-  <link name="kinect_adjust_link"/>
+  <!-- <link name="kinect_adjust_link"/>
   <joint name="kinect_adjust" type="floating">
     <origin xyz="0 0 0" rpy="0 0 0"/>
@@ -15,6 +15,7 @@
     <child link="kinect_adjust_link"/>
     <limit effort="10" lower="-0.2" upper="0.2"/>
-  </joint>
-  <xacro:sensor_kinect parent="kinect_adjust" cam_px="0.03" cam_pz="0.3" cam_or="3.14" cam_op="0.475" cam_oy="0"/>
+  </joint> -->
+  <xacro:sensor_kinect parent="base_footprint" cam_px="0.03" cam_pz="0.3" cam_or="3.14" cam_op="0.475" cam_oy="0"/>
+  <!-- <xacro:sensor_kinect parent="kinect_adjust" cam_px="0.03" cam_pz="0.3" cam_or="3.14" cam_op="0.475" cam_oy="0"/> -->
   <xacro:sensor_hokuyo parent="plate_top_link"/>
   <!-- Import manip -->

Commit message: Kinect joint and GUI
Added joint and its gui to robot decsription for camera-arm calibration
Still not tested if can run

File: all_descriptions/tgrip_description/urdf/tgrip.urdf.xacro (robot description, xacro)
@@ -9,11 +9,11 @@
   <xacro:include filename="$(find lidar_description)/urdf/hokuyo.urdf.xacro"/>
   <!--stack_hexagons parent="base_footprint"/-->
-  <!-- <link name="kinect_adjust_link"/>
+  <link name="kinect_adjust_link"/>
   <joint name="kinect_adjust" type="floating">
     <origin xyz="0 0 0" rpy="0 0 0"/>
     <parent link="base_footprint"/>
     <child link="kinect_adjust_link"/>
-    <limit effort="10" lower="-0.2" upper="0.2"/>
-  </joint> -->
+  <!--  <limit effort="10" lower="-0.2" upper="0.2"/>-->
+  </joint>
   <xacro:sensor_kinect parent="base_footprint" cam_px="0.03" cam_pz="0.3" cam_or="3.14" cam_op="0.475" cam_oy="0"/>
   <!-- <xacro:sensor_kinect parent="kinect_adjust" cam_px="0.03" cam_pz="0.3" cam_or="3.14" cam_op="0.475" cam_oy="0"/> -->

Commit message: now the om_description is correct.

File: all_descriptions/tgrip_description/urdf/tgrip.urdf.xacro (robot description, xacro)
@@ -2,5 +2,5 @@
 <robot name="tgrip" xmlns:xacro="http://ros.org/wiki/xacro">
   <xacro:include filename="$(find turtlebot_description)/urdf/turtlebot_common_library.urdf.xacro" />
-  <xacro:include filename="$(find turtlebot_description)/urdf/stacks/hexagons.urdf.xacro"/>
+  <xacro:include filename="$(find openmanipulator_description)/urdf/hexagons.urdf.xacro"/>
   <xacro:include filename="$(find turtlebot_description)/urdf/sensors/kinect.urdf.xacro"/>
   <xacro:include filename="$(find kobuki_description)/urdf/kobuki.urdf.xacro" />
@@ -8,5 +8,27 @@
   <xacro:include filename="$(find lidar_description)/urdf/hokuyo.gazebo"/>
   <xacro:include filename="$(find lidar_description)/urdf/hokuyo.urdf.xacro"/>
-  <!--stack_hexagons parent="base_footprint"/-->
+  <!-- Import manip -->
+  <!-- Import Rviz colors -->
+  <xacro:include filename="$(find open_manipulator_description)/urdf/materials.xacro" />
+  <!-- Import all Gazebo-customization elements, including Gazebo colors -->
+  <xacro:include filename="$(find open_manipulator_description)/urdf/open_manipulator.gazebo.xacro" />
+  <!-- Import Transmission -->
+  <xacro:include filename="$(find open_manipulator_description)/urdf/open_manipulator.transmission.xacro" />
+  <!-- Import URDF -->
+  <xacro:include filename="$(find open_manipulator_description)/urdf/open_manipulator.urdf.xacro" />
+  <!-- World fixed joint-->
+  <joint name="fix_world" type="fixed">
+    <origin xyz="0.16 -0.08 0.14" rpy="0 0 ${-pi/2}"/>
+    <parent link="base_footprint"/>
+    <child link="link1"/>
+  </joint>
+  <!-- Import manip -->
+  <!-- Import work space -->
+  <xacro:include filename="$(find openmanipulator_description)/urdf/open_manipulator_workspace.urdf.xacro" />
+  <!-- Workspace joint-->
+  <workspace parent="base_footprint"/>
+  <!-- Import work space -->
+  <stack_hexagons parent="base_link"/>
+  <kobuki/>
   <!-- <link name="kinect_adjust_link"/>
   <joint name="kinect_adjust" type="floating">
@@ -19,17 +41,3 @@
   <!-- <xacro:sensor_kinect parent="kinect_adjust" cam_px="0.03" cam_pz="0.3" cam_or="3.14" cam_op="0.475" cam_oy="0"/> -->
   <xacro:sensor_hokuyo parent="plate_top_link"/>
-  <!-- Import manip -->
-  <xacro:include filename="$(find open_manipulator_description)/urdf/open_manipulator_robot.urdf.xacro"/>
-  <!-- Import work space -->
-  <xacro:include filename="$(find openmanipulator_description)/urdf/open_manipulator_workspace.urdf.xacro" />
-  <!-- World fixed joint-->
-  <joint name="fix_world" type="fixed">
-    <origin xyz="0.16 -0.08 0.14" rpy="0 0 ${-pi/2}"/>
-    <parent link="base_link"/>
-    <child link="world"/>
-  </joint>
-  <!-- Workspace joint-->
-  <workspace parent="base_link"/>
-  <stack_hexagons parent="base_link"/>
-  <kobuki/>
 </robot>

File: open_manipulator/open_manipulator_description/urdf/open_manipulator.gazebo.xacro (robot description, xacro)
@@ -51,42 +51,3 @@
   </gazebo>
   <!-- camera -->
-  <gazebo reference="camera_link">
-    <sensor type="camera" name="intel_realsense_r200">
-      <update_rate>30.0</update_rate>
-      <camera name="head">
-        <horizontal_fov>1.02974</horizontal_fov>
-        <image>
-          <width>1920</width>
-          <height>1080</height>
-          <format>R8G8B8</format>
-        </image>
-        <clip>
-          <near>0.02</near>
-          <far>300</far>
-        </clip>
-        <noise>
-          <type>gaussian</type>
-          <!-- Noise is sampled independently per pixel on each frame.
-               That pixel's noise value is added to each of its color
-               channels, which at that point lie in the range [0,1]. -->
-          <mean>0.0</mean>
-          <stddev>0.007</stddev>
-        </noise>
-      </camera>
-      <plugin name="camera_controller" filename="libgazebo_ros_camera.so">
-        <alwaysOn>true</alwaysOn>
-        <updateRate>0.0</updateRate>
-        <cameraName>camera/color</cameraName>
-        <imageTopicName>image_raw</imageTopicName>
-        <cameraInfoTopicName>camera_info</cameraInfoTopicName>
-        <frameName>camera_link</frameName>
-        <hackBaseline>0.07</hackBaseline>
-        <distortionK1>0.0</distortionK1>
-        <distortionK2>0.0</distortionK2>
-        <distortionK3>0.0</distortionK3>
-        <distortionT1>0.0</distortionT1>
-        <distortionT2>0.0</distortionT2>
-      </plugin>
-    </sensor>
-  </gazebo>
 </robot>

File: open_manipulator/open_manipulator_description/urdf/open_manipulator_robot.urdf.xacro (robot description, xacro)
@@ -11,10 +11,10 @@
   <xacro:include filename="$(find open_manipulator_description)/urdf/open_manipulator.urdf.xacro" />
   <!-- World -->
-  <link name="world"/>
+  <!-- <link name="world"/> -->
   <!-- World fixed joint-->
-  <joint name="world_fixed" type="fixed">
+  <!-- <joint name="world_fixed" type="fixed">
     <origin xyz="0 0 0" rpy="0 0 0"/>
     <parent link="world"/>
     <child link="link1"/>
-  </joint>
+  </joint> -->
 </robot>

Commit message: 3DOF kinect joint
Added 3 joints: 2 prismatic and 1 continuous to calibrate kinects location
Still need to see if the axes are correct
Currently gazebo's kinect plugin doesn't work with these joints. Will either need to get rid of them post calibration or fix it somehow

File: all_descriptions/tgrip_description/urdf/tgrip.urdf.xacro (robot description, xacro)
@@ -31,13 +31,29 @@
   <stack_hexagons parent="base_link"/>
   <kobuki/>
-  <link name="kinect_adjust_link"/>
-  <joint name="kinect_adjust" type="floating">
+  <link name="kinect_adjust_link_0"/>
+  <joint name="kinect_adjust" type="continuous">
     <origin xyz="0 0 0" rpy="0 0 0"/>
+    <axis xyz="1 0 0"/>
+    <parent link="kinect_adjust_link_1"/>
+    <child link="kinect_adjust_link_0"/>
+  </joint>
+  <link name="kinect_adjust_link_1"/>
+  <joint name="kinect_adjust" type="prismatic">
+    <origin xyz="0 0 0" rpy="0 0 0"/>
+    <axis xyz="0 1 0"/>
+    <parent link="kinect_adjust_link_2"/>
+    <child link="kinect_adjust_link_1"/>
+    <limit effort="10" lower="-0.2" upper="0.2"/>-->
+  </joint>
+  <link name="kinect_adjust_link2"/>
+  <joint name="kinect_adjust" type="prismatic">
+    <origin xyz="0 0 0" rpy="0 0 0"/>
+    <axis xyz="1 0 0"/>
     <parent link="base_footprint"/>
-    <child link="kinect_adjust_link"/>
-  <!--  <limit effort="10" lower="-0.2" upper="0.2"/>-->
+    <child link="kinect_adjust_link2"/>
+    <limit effort="10" lower="-0.2" upper="0.2"/>-->
   </joint>
 <!--  <xacro:sensor_kinect parent="base_footprint" cam_px="0.03" cam_pz="0.3" cam_or="3.14" cam_op="0.475" cam_oy="0"/>-->
-  <xacro:sensor_kinect parent="kinect_adjust_link" cam_px="0.03" cam_pz="0.3" cam_or="3.14" cam_op="0.475" cam_oy="0"/>
+  <xacro:sensor_kinect parent="kinect_adjust_link_0" cam_px="0.03" cam_pz="0.3" cam_or="3.14" cam_op="0.475" cam_oy="0"/>
   <xacro:sensor_hokuyo parent="plate_top_link"/>
 </robot>

Commit message: mute the kinect_adjust joint in the tgrip.urdf.xacro

File: all_descriptions/tgrip_description/urdf/tgrip.urdf.xacro (robot description, xacro)
@@ -2,5 +2,4 @@
 <robot name="tgrip" xmlns:xacro="http://ros.org/wiki/xacro">
   <xacro:include filename="$(find turtlebot_description)/urdf/turtlebot_common_library.urdf.xacro" />
-  <xacro:include filename="$(find openmanipulator_description)/urdf/hexagons.urdf.xacro"/>
   <xacro:include filename="$(find turtlebot_description)/urdf/sensors/kinect.urdf.xacro"/>
   <xacro:include filename="$(find kobuki_description)/urdf/kobuki.urdf.xacro" />
@@ -8,4 +7,5 @@
   <xacro:include filename="$(find lidar_description)/urdf/hokuyo.gazebo"/>
   <xacro:include filename="$(find lidar_description)/urdf/hokuyo.urdf.xacro"/>
+  <xacro:include filename="$(find openmanipulator_description)/urdf/hexagons.urdf.xacro"/>
   <!-- Import manip -->
   <!-- Import Rviz colors -->
@@ -25,11 +25,11 @@
   <!-- Import manip -->
   <!-- Import work space -->
-  <xacro:include filename="$(find openmanipulator_description)/urdf/open_manipulator_workspace.urdf.xacro" />
+  <!-- <xacro:include filename="$(find openmanipulator_description)/urdf/open_manipulator_workspace.urdf.xacro" /> -->
   <!-- Workspace joint-->
-  <workspace parent="base_footprint"/>
+  <!-- <workspace parent="base_footprint"/> -->
   <!-- Import work space -->
   <stack_hexagons parent="base_link"/>
   <kobuki/>
-  <link name="kinect_adjust_link_0"/>
+  <!-- <link name="kinect_adjust_link_0"/>
   <joint name="kinect_adjust" type="continuous">
     <origin xyz="0 0 0" rpy="0 0 0"/>
@@ -37,6 +37,6 @@
     <parent link="kinect_adjust_link_1"/>
     <child link="kinect_adjust_link_0"/>
-  </joint>
-  <link name="kinect_adjust_link_1"/>
+  </joint> -->
+  <!-- <link name="kinect_adjust_link_1"/>
   <joint name="kinect_adjust" type="prismatic">
     <origin xyz="0 0 0" rpy="0 0 0"/>
@@ -44,7 +44,7 @@
     <parent link="kinect_adjust_link_2"/>
     <child link="kinect_adjust_link_1"/>
-    <limit effort="10" lower="-0.2" upper="0.2"/>-->
-  </joint>
-  <link name="kinect_adjust_link2"/>
+    <limit effort="10" lower="-0.2" upper="0.2"/>
+  </joint> -->
+  <!-- <link name="kinect_adjust_link2"/>
   <joint name="kinect_adjust" type="prismatic">
     <origin xyz="0 0 0" rpy="0 0 0"/>
@@ -52,8 +52,8 @@
     <parent link="base_footprint"/>
     <child link="kinect_adjust_link2"/>
-    <limit effort="10" lower="-0.2" upper="0.2"/>-->
-  </joint>
-<!--  <xacro:sensor_kinect parent="base_footprint" cam_px="0.03" cam_pz="0.3" cam_or="3.14" cam_op="0.475" cam_oy="0"/>-->
-  <xacro:sensor_kinect parent="kinect_adjust_link_0" cam_px="0.03" cam_pz="0.3" cam_or="3.14" cam_op="0.475" cam_oy="0"/>
+    <limit effort="10" lower="-0.2" upper="0.2"/>
+  </joint> -->
+  <xacro:sensor_kinect parent="base_footprint" cam_px="0.03" cam_pz="0.3" cam_or="3.14" cam_op="0.475" cam_oy="0"/>
+  <!-- <xacro:sensor_kinect parent="kinect_adjust_link_0" cam_px="0.03" cam_pz="0.3" cam_or="3.14" cam_op="0.475" cam_oy="0"/>  -->
   <xacro:sensor_hokuyo parent="plate_top_link"/>
 </robot>

Commit message: Kinect calibration
Adjusted constants for the fixed joint from base link to kinect
Left calibration joints commented out rather than deleting them just in case for further calibration

File: all_descriptions/tgrip_description/urdf/tgrip.urdf.xacro (robot description, xacro)
@@ -19,5 +19,5 @@
   <!-- World fixed joint-->
   <joint name="fix_world" type="fixed">
-    <origin xyz="0.16 -0.08 0.14" rpy="0 0 ${-pi/2}"/>
+    <origin xyz="0.16 -0.08 0.17" rpy="0 0 ${-pi/2}"/>
     <parent link="base_footprint"/>
     <child link="link1"/>
@@ -31,29 +31,31 @@
   <stack_hexagons parent="base_link"/>
   <kobuki/>
-  <link name="kinect_adjust_link_0"/>
-  <joint name="kinect_adjust" type="continuous">
+<!--  <link name="kinect_adjust_link_2"/>
+  <joint name="kinect_adjust_2" type="continuous">
+    <origin xyz="0 0 0" rpy="0 0 0"/>
+    <axis xyz="0 1 0"/>
+    <parent link="kinect_adjust_link_1"/>
+    <child link="kinect_adjust_link_2"/>
+    <limit velocity="1.0" effort="10" lower="-0.2" upper="0.2"/>
+  </joint>
+  <link name="kinect_adjust_link_1"/>
+  <joint name="kinect_adjust_1" type="prismatic">
     <origin xyz="0 0 0" rpy="0 0 0"/>
     <axis xyz="1 0 0"/>
-    <parent link="kinect_adjust_link_1"/>
-    <child link="kinect_adjust_link_0"/>
+    <parent link="kinect_adjust_link_0"/>
+    <child link="kinect_adjust_link_1"/>
+    <limit velocity="1.0" effort="10" lower="-0.2" upper="0.2"/>
   </joint>
-  <link name="kinect_adjust_link_1"/>
-  <joint name="kinect_adjust" type="prismatic">
+  <link name="kinect_adjust_link_0"/>
+  <joint name="kinect_adjust_0" type="prismatic">
     <origin xyz="0 0 0" rpy="0 0 0"/>
     <axis xyz="0 1 0"/>
-    <parent link="kinect_adjust_link_2"/>
-    <child link="kinect_adjust_link_1"/>
-    <limit effort="10" lower="-0.2" upper="0.2"/>-->
+    <parent link="base_link"/>
+    <child link="kinect_adjust_link_0"/>
+    <limit velocity="1.0" effort="10" lower="-0.2" upper="0.2"/>
   </joint>
-  <link name="kinect_adjust_link2"/>
-  <joint name="kinect_adjust" type="prismatic">
-    <origin xyz="0 0 0" rpy="0 0 0"/>
-    <axis xyz="1 0 0"/>
-    <parent link="base_footprint"/>
-    <child link="kinect_adjust_link2"/>
-    <limit effort="10" lower="-0.2" upper="0.2"/>-->
-  </joint>
+  -->
 <!--  <xacro:sensor_kinect parent="base_footprint" cam_px="0.03" cam_pz="0.3" cam_or="3.14" cam_op="0.475" cam_oy="0"/>-->
-  <xacro:sensor_kinect parent="kinect_adjust_link_0" cam_px="0.03" cam_pz="0.3" cam_or="3.14" cam_op="0.475" cam_oy="0"/>
+  <xacro:sensor_kinect parent="base_link" cam_px="-0.015" cam_py="0.04" cam_pz="0.3" cam_or="3.14" cam_op="0.475" cam_oy="0"/>
   <xacro:sensor_hokuyo parent="plate_top_link"/>
 </robot>

Commit message: To solve the om description and the plugin conflict, I fixed every joint of the om. So it's a rigid body on the turtlebot base now, and the navigation is good to go.

File: all_descriptions/tgrip_description/urdf/tgrip.urdf.xacro (robot description, xacro)
@@ -25,7 +25,7 @@
   <!-- Import manip -->
   <!-- Import work space -->
-  <!-- <xacro:include filename="$(find openmanipulator_description)/urdf/open_manipulator_workspace.urdf.xacro" /> -->
+  <xacro:include filename="$(find openmanipulator_description)/urdf/open_manipulator_workspace.urdf.xacro" />
   <!-- Workspace joint-->
-  <!-- <workspace parent="base_footprint"/> -->
+  <workspace parent="base_footprint"/>
   <!-- Import work space -->
   <stack_hexagons parent="base_link"/>

File: open_manipulator/open_manipulator_description/urdf/open_manipulator.gazebo.xacro (robot description, xacro)
@@ -34,5 +34,5 @@
   </gazebo>
   <!-- ros_control plugin -->
-  <gazebo>
+  <!-- <gazebo>
     <plugin name="gazebo_ros_control" filename="libgazebo_ros_control.so">
       <controlPeriod>0.001</controlPeriod>
@@ -40,7 +40,7 @@
       <legacyModeNS>true</legacyModeNS>
     </plugin>
-  </gazebo>
-  <gazebo>
-    <!-- loading plugin: mimic joints works in gazebo now -->
+  </gazebo> -->
+  <!-- loading plugin: mimic joints works in gazebo now -->
+  <!-- <gazebo>
     <plugin name="gazebo_gripper_ros_control" filename="libroboticsgroup_gazebo_mimic_joint_plugin.so">
       <joint>gripper</joint>
@@ -49,5 +49,5 @@
       <offset>0.0</offset>
     </plugin>
-  </gazebo>
+  </gazebo> -->
   <!-- camera -->
 </robot>

File: open_manipulator/open_manipulator_description/urdf/open_manipulator.urdf.xacro (robot description, xacro)
@@ -17,4 +17,5 @@
       </geometry>
     </collision>
+  <!-- The regular expression "-?\d.\d{7}e-0[0-9]" -->
     <inertial>
       <origin xyz="3.0876154e-04 0.0000000e+00 -1.2176461e-04" />
@@ -26,5 +27,5 @@
   </link>
   <!-- Joint 1 -->
-  <joint name="joint1" type="revolute">
+  <joint name="joint1" type="fixed">
     <parent link="link1"/>
     <child link="link2"/>
@@ -57,5 +58,5 @@
   </link>
   <!--  Joint 2 -->
-  <joint name="joint2" type="revolute">
+  <joint name="joint2" type="fixed">
     <parent link="link2"/>
     <child link="link3"/>
@@ -88,5 +89,5 @@
   </link>
   <!--  Joint 3 -->
-  <joint name="joint3" type="revolute">
+  <joint name="joint3" type="fixed">
     <parent link="link3"/>
     <child link="link4"/>
@@ -119,5 +120,5 @@
   </link>
   <!--  Joint 4 -->
-  <joint name="joint4" type="revolute">
+  <joint name="joint4" type="fixed">
     <parent link="link4"/>
     <child link="link5"/>
@@ -150,5 +151,5 @@
   </link>
   <!--  Gripper joint -->
-  <joint name="gripper" type="prismatic">
+  <joint name="gripper" type="fixed">
     <parent link="link5"/>
     <child link="gripper_link"/>
@@ -181,5 +182,5 @@
   </link>
   <!--  Gripper joint sub -->
-  <joint name="gripper_sub" type="prismatic">
+  <joint name="gripper_sub" type="fixed">
     <parent link="link5"/>
     <child link="gripper_link_sub"/>

Commit message: om description for nav

File: all_descriptions/tgrip_description/urdf/tgrip.urdf.xacro (robot description, xacro)
@@ -19,9 +19,13 @@
   <!-- World fixed joint-->
   <joint name="fix_world" type="fixed">
-    <origin xyz="0.16 -0.08 0.14" rpy="0 0 ${-pi/2}"/>
-    <parent link="base_footprint"/>
+    <origin xyz="0.16 -0.08 0.17" rpy="0 0 ${-pi/2}"/>
+    <parent link="base_link"/>
     <child link="link1"/>
   </joint>
   <!-- Import manip -->
+<!-- for nav module -->
+  <!-- <xacro:include filename="$(find openmanipulator_description)/urdf/open_manipulator_nav.urdf.xacro" /> -->
+  <!-- <xacro:include filename="$(find open_manipulator_description)/urdf/open_manipulator.gazebo.xacro" /> -->
+<!-- for nav module -->
   <!-- Import work space -->
   <xacro:include filename="$(find openmanipulator_description)/urdf/open_manipulator_workspace.urdf.xacro" />
@@ -31,13 +35,13 @@
   <stack_hexagons parent="base_link"/>
   <kobuki/>
-  <link name="kinect_adjust_link"/>
+  <!-- <link name="kinect_adjust_link"/>
   <joint name="kinect_adjust" type="floating">
     <origin xyz="0 0 0" rpy="0 0 0"/>
     <parent link="base_footprint"/>
     <child link="kinect_adjust_link"/>
-  <!--  <limit effort="10" lower="-0.2" upper="0.2"/>-->
-  </joint>
-<!--  <xacro:sensor_kinect parent="base_footprint" cam_px="0.03" cam_pz="0.3" cam_or="3.14" cam_op="0.475" cam_oy="0"/>-->
-  <xacro:sensor_kinect parent="kinect_adjust_link" cam_px="0.03" cam_pz="0.3" cam_or="3.14" cam_op="0.475" cam_oy="0"/>
+   <limit effort="10" lower="-0.2" upper="0.2"/>
+  </joint> -->
+ <xacro:sensor_kinect parent="base_footprint" cam_px="0.03" cam_pz="0.3" cam_or="3.14" cam_op="0.475" cam_oy="0"/>
+  <!-- <xacro:sensor_kinect parent="kinect_adjust_link" cam_px="0.03" cam_pz="0.3" cam_or="3.14" cam_op="0.475" cam_oy="0"/>  -->
   <xacro:sensor_hokuyo parent="plate_top_link"/>
 </robot>
