Commit message: roll back to original urdf

File: open_manipulator/open_manipulator_description/urdf/open_manipulator.gazebo.xacro (robot description, xacro)
@@ -34,5 +34,5 @@
   </gazebo>
   <!-- ros_control plugin -->
-  <!-- <gazebo>
+  <gazebo>
     <plugin name="gazebo_ros_control" filename="libgazebo_ros_control.so">
       <controlPeriod>0.001</controlPeriod>
@@ -40,7 +40,7 @@
       <legacyModeNS>true</legacyModeNS>
     </plugin>
-  </gazebo> -->
+  </gazebo>
   <!-- loading plugin: mimic joints works in gazebo now -->
-  <!-- <gazebo>
+  <gazebo>
     <plugin name="gazebo_gripper_ros_control" filename="libroboticsgroup_gazebo_mimic_joint_plugin.so">
       <joint>gripper</joint>
@@ -49,5 +49,5 @@
       <offset>0.0</offset>
     </plugin>
-  </gazebo> -->
+  </gazebo>
   <!-- camera -->
 </robot>

File: open_manipulator/open_manipulator_description/urdf/open_manipulator.urdf.xacro (robot description, xacro)
@@ -17,5 +17,4 @@
       </geometry>
     </collision>
-  <!-- The regular expression "-?\d.\d{7}e-0[0-9]" -->
     <inertial>
       <origin xyz="3.0876154e-04 0.0000000e+00 -1.2176461e-04" />
@@ -27,5 +26,5 @@
   </link>
   <!-- Joint 1 -->
-  <joint name="joint1" type="fixed">
+  <joint name="joint1" type="revolute">
     <parent link="link1"/>
     <child link="link2"/>
@@ -58,5 +57,5 @@
   </link>
   <!--  Joint 2 -->
-  <joint name="joint2" type="fixed">
+  <joint name="joint2" type="revolute">
     <parent link="link2"/>
     <child link="link3"/>
@@ -89,5 +88,5 @@
   </link>
   <!--  Joint 3 -->
-  <joint name="joint3" type="fixed">
+  <joint name="joint3" type="revolute">
     <parent link="link3"/>
     <child link="link4"/>
@@ -120,5 +119,5 @@
   </link>
   <!--  Joint 4 -->
-  <joint name="joint4" type="fixed">
+  <joint name="joint4" type="revolute">
     <parent link="link4"/>
     <child link="link5"/>
@@ -151,5 +150,5 @@
   </link>
   <!--  Gripper joint -->
-  <joint name="gripper" type="fixed">
+  <joint name="gripper" type="prismatic">
     <parent link="link5"/>
     <child link="gripper_link"/>
@@ -182,5 +181,5 @@
   </link>
   <!--  Gripper joint sub -->
-  <joint name="gripper_sub" type="fixed">
+  <joint name="gripper_sub" type="prismatic">
     <parent link="link5"/>
     <child link="gripper_link_sub"/>
@@ -220,5 +219,5 @@
   </joint>
   <!-- end effector link -->
-  <link name="end_effector_link">
+  <!-- <link name="end_effector_link">
     <visual>
       <origin xyz="0 0 0" rpy="0 0 0"/>
@@ -235,7 +234,7 @@
                izz="1.0e-03" />
     </inertial>
-  </link>
-  <!-- Realsense Camera Joint Position
-  <joint name="camera_joint" type="fixed">
+  </link> -->
+  <!-- Realsense Camera Joint Position -->
+  <!-- <joint name="camera_joint" type="fixed">
     <axis xyz="0 1 0" />
     <origin xyz="0.070 0.032 0.052" rpy="0 0 0"/>
